File: hardware/amp_green_island/preamp_ch1.kicad_sch (KiCad schematic)
At the start: 30 parts, among them U101 OP27, U102 TL072

Commit message: amp_green_island: add all 4 channels to schematic
Parts:
- renumbered C104 to C101, C105 to C102, C109 to C103, C101 to C104, C102 to C105, C103 to C106, C106 to C107, C107 to C108, C108 to C109, R104 to R103, R105 to R104, R106 to R105, R107 to R106, R109 to R107, R110 to R108, R111 to R109, R112 to R110, R113 to R111, R114 to R112, R115 to R113, R116 to R114
Other:
- moved on the sheet: C101, C102, C103, C104, C105, C106, C107, C108, C109, D101, D102, R101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

Commit message: amp_green_island: pcb verified
Parts:
- U102: footprint Package_SO:SOIC-8-1EP_3.9x4.9mm_P1.27mm_EP2.41x3.81mm_ThermalVias -> Package_SO:SO-8_3.9x4.9mm_P1.27mm
Changed lines of the file:
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@@
       (effects (font (size 1.27 1.27)))
     )
-    (property "Footprint" "Package_SO:SOIC-8-1EP_3.9x4.9mm_P1.27mm_EP2.41x3.81mm_ThermalVias" (at 187.96 88.9 0)
+    (property "Footprint" "Package_SO:SO-8_3.9x4.9mm_P1.27mm" (at 187.96 88.9 0)
       (effects (font (size 1.27 1.27)) hide)
     )
@@
       (effects (font (size 1.27 1.27)) (justify left))
     )
-    (property "Footprint" "Package_SO:SOIC-8-1EP_3.9x4.9mm_P1.27mm_EP2.41x3.81mm_ThermalVias" (at 184.15 59.69 0)
+    (property "Footprint" "Package_SO:SO-8_3.9x4.9mm_P1.27mm" (at 184.15 59.69 0)
       (effects (font (size 1.27 1.27)) hide)
     )
@@
       (effects (font (size 1.27 1.27)))
     )
-    (property "Footprint" "Package_SO:SOIC-8-1EP_3.9x4.9mm_P1.27mm_EP2.41x3.81mm_ThermalVias" (at 143.51 86.36 0)
-      (effects (font (size 1.27 1.27)) hide)
-    )
+    (property "Footprint" "Package_SO:SO-8_3.9x4.9mm_P1.27mm" (at 143.51 86.36 0)
+      (effects (font (size 1.27 1.27)) hide)
+    )
