File: hardware/amp_green_island/preamp_ch4.kicad_sch (KiCad schematic)
At the start: 0 parts

Commit message: amp_green_island: add all 4 channels to schematic
Parts:
- added C101, C102, C106, C107: 100n, Capacitor_SMD:C_0805_2012Metric_Pad1.18x1.45mm_HandSolder, symbol Device:C
- added C103, C108: 100n, Capacitor_THT:C_Rect_L7.2mm_W4.5mm_P5.00mm_FKS2_FKP2_MKS2_MKP2, symbol Device:C
- added C104, C105, C109: 1u, Capacitor_THT:C_Rect_L7.2mm_W7.2mm_P5.00mm_FKS2_FKP2_MKS2_MKP2, symbol Device:C
- added D101, D102: LL4148, Diode_SMD:D_MiniMELF, symbol Diode:LL4148
- added R101, R102: 10k, Resistor_SMD:R_0805_2012Metric_Pad1.20x1.40mm_HandSolder, symbol Device:R
- added R104, R105: 100k, Resistor_SMD:R_0805_2012Metric_Pad1.20x1.40mm_HandSolder, symbol Device:R
- added R106, R110: 1k, Resistor_SMD:R_0805_2012Metric_Pad1.20x1.40mm_HandSolder, symbol Device:R
- added R107: 200k, Resistor_SMD:R_MiniMELF_MMA-0204, symbol Device:R
- added R109: 3k3, Resistor_SMD:R_MiniMELF_MMA-0204, symbol Device:R
- added R111: 5k6, Resistor_SMD:R_0805_2012Metric_Pad1.20x1.40mm_HandSolder, symbol Device:R
- added R112: 82k, Resistor_SMD:R_0805_2012Metric_Pad1.20x1.40mm_HandSolder, symbol Device:R
- added R113, R116: 470, Resistor_SMD:R_MELF_MMB-0207, symbol Device:R
- added R114, R115: 33k, Resistor_SMD:R_MELF_MMB-0207, symbol Device:R
- added RV101: 10k, Potentiometer_SMD:Potentiometer_Bourns_3314G_Vertical, symbol Device:R_Potentiometer
- added RV102: 50k, Potentiometer_SMD:Potentiometer_Bourns_3314G_Vertical, symbol Device:R_Potentiometer
- added RV103: 5k, Potentiometer_SMD:Potentiometer_Bourns_3314G_Vertical, symbol Device:R_Potentiometer
- added U101: OP27, Package_SO:SO-8_3.9x4.9mm_P1.27mm, symbol pff_ic:LT1677
- added U102: TL072, Package_SO:SOIC-8-1EP_3.9x4.9mm_P1.27mm_EP2.41x3.81mm_ThermalVias, symbol Amplifier_Operational:TL072
Connections:
- new net: C104.2, R102.2, R104.2, U101.3 (+)
- new net: R109.2, R111.1, R112.1, U102.6 (-)
- new net: D101.2 (A), D102.1 (K), R113.2, R116.1
- new net: R115.1, RV103.1
- new net: R111.2, RV102.1
- new net: R113.1, RV102.2, RV102.3, U102.7
- new net: R112.2, RV103.2
- new net: R114.2, RV103.3
- new net: RV101.1, U101.1 (TRIM1)
- new net: RV101.3, U101.8 (TRIM8)
- new net: C109.2, R107.2, R110.1, U102.1
- new net: C109.1, R106.2, R107.1, U102.2 (-)
- new net: R110.2, U102.5 (+)
- new net: C105.1, R101.2, R105.2, U101.2 (-)
- new net: C105.2, R105.1, R106.1, U101.6
- new net +12V: C101.1, C102.1, C103.1, D101.1 (K), R114.1, RV101.2, U101.7 (V+), U102.8 (V+)
- new net -12V: C106.1, C107.1, C108.1, D102.2 (A), R115.2, U101.4 (V-), U102.4 (V-)
- new net GND: C101.2, C102.2, C103.2, C104.1, C106.2, C107.2, C108.2, R104.1, R109.1, U102.3 (+)
- new net in4_+: R102.1
- new net in4_-: R101.1
- new net out4: R116.2
Other:
- note added: "0v trim"
- note added: "gain"
- note added: "offset"

Commit message: amp_green_island: pcb verified
Parts:
- U102: footprint Package_SO:SOIC-8-1EP_3.9x4.9mm_P1.27mm_EP2.41x3.81mm_ThermalVias -> Package_SO:SO-8_3.9x4.9mm_P1.27mm
Changed lines of the file:
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@@
       (effects (font (size 1.27 1.27)))
     )
-    (property "Footprint" "Package_SO:SOIC-8-1EP_3.9x4.9mm_P1.27mm_EP2.41x3.81mm_ThermalVias" (at 151.13 83.82 0)
+    (property "Footprint" "Package_SO:SO-8_3.9x4.9mm_P1.27mm" (at 151.13 83.82 0)
       (effects (font (size 1.27 1.27)) hide)
     )
@@
       (effects (font (size 1.27 1.27)))
     )
-    (property "Footprint" "Package_SO:SOIC-8-1EP_3.9x4.9mm_P1.27mm_EP2.41x3.81mm_ThermalVias" (at 195.58 86.36 0)
+    (property "Footprint" "Package_SO:SO-8_3.9x4.9mm_P1.27mm" (at 195.58 86.36 0)
       (effects (font (size 1.27 1.27)) hide)
     )
@@
       (effects (font (size 1.27 1.27)) (justify left))
     )
-    (property "Footprint" "Package_SO:SOIC-8-1EP_3.9x4.9mm_P1.27mm_EP2.41x3.81mm_ThermalVias" (at 191.77 57.15 0)
-      (effects (font (size 1.27 1.27)) hide)
-    )
+    (property "Footprint" "Package_SO:SO-8_3.9x4.9mm_P1.27mm" (at 191.77 57.15 0)
+      (effects (font (size 1.27 1.27)) hide)
+    )
